Commit message: Dual-hand Manus glove -> Allegro retargeting for a bimanual UR3/UR3e torso
- left Allegro: mirrored URDF, allegro_left config with per-joint sign/offset (applied in env/hand.py)
- Manus ROS 2 clients for both gloves, left-hand keypoint FK, session recorder
- dual-hand runtime: geort_streamer_dual (ZMQ) + ros_joint_bridge_dual (ROS 2 JointState), run_dual_teleop.sh
- trained models (config + last.pth per run) and FK models; 400 training epochs
- flexion-correlation evaluation, replay renderer, project page and README
- rule-based baseline: dex2all + dexhand_manus patch + pinned upstream packages
- requirements: pin sapien==2.2.2 and numpy<2 (SAPIEN 3 breaks env/hand.py)

File: assets/allegro_left/allegro_hand_left.urdf (robot description, URDF)
Before this commit: robot allegro_left, 23 links, 22 joints
Links:
- link link_0.0: mass 0.0119 -> 0.005
- link link_11.0: mass 0.0096 -> 0.02
- link link_3.0: mass 0.02 -> 0.0096
- link link_8.0: mass 0.005 -> 0.0119
Joints:
- joint joint_0.0: origin xyz=0 0.0435 -0.001542 rpy=-0.08726646255 0 0 -> xyz=0 -0.0435 -0.001542 rpy=0.08726646255 0 0
- joint joint_8.0: origin xyz=0 -0.0435 -0.001542 rpy=0.08726646255 0 0 -> xyz=0 0.0435 -0.001542 rpy=-0.08726646255 0 0
